File: pcb/pcb.kicad_pcb (KiCad board)
At the start: 2 copper layers, 60 x 35 mm, 20 parts, among them J1 Conn_01x09_Pin, J2 Conn_01x09_Pin, J3 Conn_01x09_Pin, J4 Conn_01x09_Pin, J5 Conn_01x04_Pin, J6 Conn_01x04_Pin, J9 Conn_01x09_Pin

Commit message: chore: annotation cleanup
Parts:
- J1, J3, J4, J9: value Conn_01x09_Pin -> Pin1x9
- J2: value Conn_01x09_Pin -> Pin1x4
- J5, J6: value Conn_01x04_Pin -> Pin1x4
- moved R9 0.10 mm to (37.9, 43.4)
