File: pcb/pcb.kicad_sch (KiCad schematic)
At the start: 30 parts, among them J1 Conn_01x09_Pin, J2 Conn_01x09_Pin, J3 Conn_01x09_Pin, J4 Conn_01x09_Pin, SW1 SW_Push, SW2 SW_Push, SW3 SW_Push, SW4 SW_Push, SW5 SW_Push

Commit message: feat: completion of pcb
Parts:
- added J10: Conn_01x09_Pin, symbol Connector:Conn_01x09_Pin
- added J5, J6: Conn_01x04_Pin, Connector_PinSocket_2.54mm:PinSocket_1x04_P2.54mm_Vertical, symbol Connector:Conn_01x04_Pin
- added J7, J8: Conn_01x04_Pin, symbol Connector:Conn_01x04_Pin
- added J9: Conn_01x09_Pin, Connector_PinSocket_2.54mm:PinSocket_1x09_P2.54mm_Vertical_SMD_Pin1Left, symbol Connector:Conn_01x09_Pin
- added SW6: SW_Push, symbol Switch:SW_Push
- J1, J2, J3, J4: footprint (none) -> Connector_PinHeader_2.54mm:PinHeader_1x09_P2.54mm_Vertical
Connections:
- net +3V3: now also J5.1 (Pin_1), J6.1 (Pin_1); no longer SW1.2, SW2.2, SW3.2, SW4.2, SW5.2
- net B.11: now also R10.2; no longer D5.2 (A)
- net B.14: now also R9.2; no longer D4.2 (A)
- net B.17: now also R8.2; no longer D3.2 (A)
- net B.2: now also R13.2; no longer D8.2 (A)
- net B.20: now also R7.2; no longer D2.2 (A)
- net B.21: now also R6.2; no longer D1.2 (A)
- net B.5: now also R12.2; no longer D7.2 (A)
- net B.8: now also R11.2; no longer D6.2 (A)
- net GND: now also D1.1 (K), D2.1 (K), D3.1 (K), D4.1 (K), D5.1 (K), D6.1 (K), D7.1 (K), D8.1 (K), J10.1 (Pin_1), J9.1 (Pin_1); no longer R10.1, R11.1, R12.1, R13.1, R6.1, R7.1, R8.1, R9.1
- net at SW5.1: now also J8.3 (Pin_3); no longer R5.2
- net at SW1.1: now also J7.2 (Pin_2); no longer R1.2
- net at SW4.1: now also J8.2 (Pin_2); no longer R4.2
- net at SW2.1: now also J7.3 (Pin_3); no longer R2.2
- net at SW3.1: now also J7.4 (Pin_4); no longer R3.2
- new net: J9.7 (Pin_7), R11.1
- new net: J9.8 (Pin_8), R12.1
- new net: D1.2 (A), J10.2 (Pin_2)
- new net: J9.9 (Pin_9), R13.1
- new net: D4.2 (A), J10.5 (Pin_5)
- new net: J9.2 (Pin_2), R6.1
- new net: D3.2 (A), J10.4 (Pin_4)
- new net: J8.4 (Pin_4), SW6.1
- new net: J9.6 (Pin_6), R10.1
- new net: J5.2 (Pin_2), J6.2 (Pin_2), R1.2
- new net: J6.3 (Pin_3), R4.2
- new net: J6.4 (Pin_4), R5.2
- new net: D2.2 (A), J10.3 (Pin_3)
- new net: J9.3 (Pin_3), R7.1
- new net: J9.4 (Pin_4), R8.1
- new net: J9.5 (Pin_5), R9.1
- new net: J5.4 (Pin_4), R3.2
- new net: D5.2 (A), J10.6 (Pin_6)
- new net: D6.2 (A), J10.7 (Pin_7)
- new net: J5.3 (Pin_3), R2.2
- new net: D8.2 (A), J10.9 (Pin_9)
- new net: D7.2 (A), J10.8 (Pin_8)
- new net VCC: J7.1 (Pin_1), J8.1 (Pin_1), SW1.2, SW2.2, SW3.2, SW4.2, SW5.2, SW6.2
Other:
- note added: "Controller 1"
- note added: "Controller 2"
- moved on the sheet: D1, D2, D3, D4, D5, D6, D7, D8, R10, R11, R12, R13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

Commit message: feat: completion of pcb routing
Parts:
- J5, J6: footprint Connector_PinSocket_2.54mm:PinSocket_1x04_P2.54mm_Vertical -> Connector_PinHeader_2.54mm:PinHeader_1x04_P2.54mm_Vertical
- J9: footprint Connector_PinSocket_2.54mm:PinSocket_1x09_P2.54mm_Vertical_SMD_Pin1Left -> Connector_PinHeader_2.54mm:PinHeader_1x09_P2.54mm_Vertical
- R1, R10, R11, R12, R13, R2, R3, R4, R5, R6, R7, R8, R9: footprint (none) -> Resistor_THT:R_Axial_DIN0207_L6.3mm_D2.5mm_P10.16mm_Horizontal
Changed lines of the file:
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@@
 			)
 		)
-		(property "Footprint" ""
+		(property "Footprint" "Resistor_THT:R_Axial_DIN0207_L6.3mm_D2.5mm_P10.16mm_Horizontal"
 			(at 83.82 135.128 90)
 			(hide yes)
@@
 			)
 		)
-		(property "Footprint" ""
+		(property "Footprint" "Resistor_THT:R_Axial_DIN0207_L6.3mm_D2.5mm_P10.16mm_Horizontal"
 			(at 83.82 141.478 90)
 			(hide yes)
@@
 			)
 		)
-		(property "Footprint" ""
+		(property "Footprint" "Resistor_THT:R_Axial_DIN0207_L6.3mm_D2.5mm_P10.16mm_Horizontal"
 			(at 83.82 147.828 90)
 			(hide yes)
@@
 			)
 		)
-		(property "Footprint" ""
+		(property "Footprint" "Resistor_THT:R_Axial_DIN0207_L6.3mm_D2.5mm_P10.16mm_Horizontal"
 			(at 83.82 103.378 90)
 			(hide yes)
@@
 			)
 		)
-		(property "Footprint" ""
+		(property "Footprint" "Resistor_THT:R_Axial_DIN0207_L6.3mm_D2.5mm_P10.16mm_Horizontal"
 			(at 83.82 128.778 90)
 			(hide yes)
@@
 			)
 		)
-		(property "Footprint" "Connector_PinSocket_2.54mm:PinSocket_1x04_P2.54mm_Vertical"
+		(property "Footprint" "Connector_PinHeader_2.54mm:PinHeader_1x04_P2.54mm_Vertical"
 			(at 160.02 60.96 0)
 			(hide yes)
@@
 			)
 		)
-		(property "Footprint" ""
+		(property "Footprint" "Resistor_THT:R_Axial_DIN0207_L6.3mm_D2.5mm_P10.16mm_Horizontal"
 			(at 135.89 65.278 90)
 			(hide yes)
@@
 			)
 		)
-		(property "Footprint" "Connector_PinSocket_2.54mm:PinSocket_1x09_P2.54mm_Vertical_SMD_Pin1Left"
+		(property "Footprint" "Connector_PinHeader_2.54mm:PinHeader_1x09_P2.54mm_Vertical"
 			(at 66.04 109.22 0)
 			(hide yes)
@@
 			)
 		)
-		(property "Footprint" ""
+		(property "Footprint" "Resistor_THT:R_Axial_DIN0207_L6.3mm_D2.5mm_P10.16mm_Horizontal"
 			(at 83.82 109.728 90)
 			(hide yes)
@@
 			)
 		)
-		(property "Footprint" ""
+		(property "Footprint" "Resistor_THT:R_Axial_DIN0207_L6.3mm_D2.5mm_P10.16mm_Horizontal"
 			(at 135.89 44.958 90)
 			(hide yes)
@@
 			)
 		)
-		(property "Footprint" ""
+		(property "Footprint" "Resistor_THT:R_Axial_DIN0207_L6.3mm_D2.5mm_P10.16mm_Horizontal"
 			(at 135.89 39.878 90)
 			(hide yes)
@@
 			)
 		)
-		(property "Footprint" ""
+		(property "Footprint" "Resistor_THT:R_Axial_DIN0207_L6.3mm_D2.5mm_P10.16mm_Horizontal"
 			(at 135.89 70.358 90)
 			(hide yes)
@@
 			)
 		)
-		(property "Footprint" "Connector_PinSocket_2.54mm:PinSocket_1x04_P2.54mm_Vertical"
+		(property "Footprint" "Connector_PinHeader_2.54mm:PinHeader_1x04_P2.54mm_Vertical"
 			(at 160.02 25.4 0)
 			(hide yes)
@@
 			)
 		)
-		(property "Footprint" ""
+		(property "Footprint" "Resistor_THT:R_Axial_DIN0207_L6.3mm_D2.5mm_P10.16mm_Horizontal"
 			(at 135.89 27.178 90)
 			(hide yes)
@@
 			)
 		)
-		(property "Footprint" ""
+		(property "Footprint" "Resistor_THT:R_Axial_DIN0207_L6.3mm_D2.5mm_P10.16mm_Horizontal"
 			(at 83.82 116.078 90)
 			(hide yes)
@@
 			)
 		)
-		(property "Footprint" ""
+		(property "Footprint" "Resistor_THT:R_Axial_DIN0207_L6.3mm_D2.5mm_P10.16mm_Horizontal"
 			(at 83.82 122.428 90)
 			(hide yes)

Commit message: chore: annotation cleanup
Parts:
- J1, J10, J3, J4, J9: value Conn_01x09_Pin -> Pin1x9
- J2: value Conn_01x09_Pin -> Pin1x4; footprint Connector_PinHeader_2.54mm:PinHeader_1x09_P2.54mm_Vertical -> Connector_PinHeader_2.54mm:PinHeader_1x04_P2.54mm_Vertical
- J5, J6, J7, J8: value Conn_01x04_Pin -> Pin1x4
Other:
- moved on the sheet: D1, D2, D3, D4, D5, D6, D7, D8, J10
